File: PCB_designes/KiCad_PCB_design/Arduino_Relay/Arduino_relay/Arduino_relay.kicad_pcb (KiCad board)
At the start: 2 copper layers, 116 parts, among them J1 Mains_Power, J10 DHT11, J11 LED_A, J12 LED_K, J15 I2C_LCD, J2 Plant_Motor, J3 Mist_Motor, J4 Bucket_Motor, J5 Lights, J6 Sensor_2, J7 Sensor_1, K1 FINDER-36.11, K2 FINDER-36.11, K3 FINDER-36.11, K4 FINDER-36.11, Q1 BC547, Q2 BC547, Q3 BC547, Q4 BC547, U4 SFH617A-1, U5 SFH617A-1, U6 SFH617A-1, U7 SFH617A-1

Commit message: Added Images
Parts:
- removed the A1 at (128.3, 70.4)
- removed the D1 at (190.6, 46.2)
- removed the D2 at (211.4, 46.4)
- removed the D3 at (150.4, 45.5)
- removed the D4 at (169.6, 45.8)
- removed the J1 at (231.2, 29.0)
- removed the J10 at (133.6, 54.8)
- removed the J11 at (133.4, 41.0)
- removed the J12 at (133.8, 66.3)
- removed the J15 at (123.2, 27.0)
- removed the J2 at (215.9, 73.0)
- removed the J3 at (194.5, 72.8)
- removed the J4 at (173.3, 72.8)
- removed the J5 at (154.0, 72.6)
- removed the J6 at (103.2, 54.6)
- removed the J7 at (106.7, 40.0)
- removed the K1 at (216.6, 50.3)
- removed the K2 at (195.6, 50.2)
- removed the K3 at (174.7, 50.3)
- removed the K4 at (155.6, 50.1)
- removed the Q1 at (221.8, 41.2)
- removed the Q2 at (201.6, 40.6)
- removed the Q3 at (181.4, 40.2)
- removed the Q4 at (162.4, 39.6)
- removed the R1 at (215.7, 37.2)
- removed the R11 at (117.3, 50.1)
- removed the R12 at (117.5, 58.6)
- removed the R13 at (117.5, 61.4)
- removed the R14 at (117.3, 42.5)
- removed the R15 at (117.3, 45.0)
- removed the R16 at (117.3, 47.5)
- removed the R17 at (138.9, 65.4)
- removed the R18 at (138.9, 68.5)
- removed the R19 at (138.9, 71.4)
- removed the R2 at (195.5, 36.0)
- removed the R20 at (138.9, 74.4)
- removed the R3 at (174.7, 34.0)
- removed the R4 at (154.5, 33.8)
- removed the R5 at (215.6, 40.8)
- removed the R6 at (195.5, 40.0)
- removed the R7 at (174.7, 39.6)
- removed the R8 at (154.7, 39.6)
- removed the TP1 at (157.4, 42.2)
- removed the TP15 at (110.2, 32.0)
- removed the TP16 at (109.6, 55.2)
- removed the TP17 at (117.4, 52.6)
- removed the TP18 at (117.2, 39.0)
- removed the TP2 at (204.2, 42.8)
- removed the TP3 at (164.8, 42.2)
- removed the TP4 at (175.6, 42.4)
- removed the TP5 at (184.4, 42.4)
- removed the TP6 at (196.2, 42.8)
- removed the TP7 at (124.6, 52.6)
- removed the TP8 at (124.6, 63.2)
- removed the U4 at (211.8, 35.0)
- removed the U5 at (191.3, 34.2)
- removed the U6 at (170.6, 34.2)
- removed the U7 at (150.4, 34.4)
Routing:
- net (no net): track 1405.5 -> 0.00 mm
- removed copper zone on B.Cu, net (none)
