File: PCB_designes/KiCad_PCB_design/Arduino_Relay/Arduino_relay/Arduino_relay.sch (KiCad schematic (older format))
At the start: 58 parts, among them J1 Mains_Power, J10 DHT11, J11 LED_A, J12 LED_K, J15 I2C_LCD, J2 Plant_Motor, J3 Mist_Motor, J4 Bucket_Motor, J5 Lights, J6 Sensor_2, J7 Sensor_1, K1 FINDER-36.11, K2 FINDER-36.11, K3 FINDER-36.11, K4 FINDER-36.11, Q1 BC547, Q2 BC547, Q3 BC547, Q4 BC547, U4 SFH617A-1, U5 SFH617A-1, U6 SFH617A-1, U7 SFH617A-1

Commit message: Added Images
Other:
- moved on the sheet: A1, D1, D2, D3, D4, J10, J11, J12, J2, J3, J4, J5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
