File: PCB_designes/KiCad_PCB_design/ESP_PCB/ESP_PCB/ESP_PCB.kicad_pcb (KiCad board)
At the start: 2 copper layers, 26 parts, among them J1 Pwr, J2 LCD_Connector, J3 I2C_2, J4 Rotary_Encoder, J5 I2C_1, J6 I2C_3, U1 AT24C512, U2 DS1307_RTC, U3 ESP32_dev

Commit message: Added Images
Parts:
- removed the C1 at (248.2, 88.5)
- removed the C2 at (246.0, 85.5)
- removed the J1 at (258.8, 91.5)
- removed the J2 at (259.8, 120.1)
- removed the J3 at (238.5, 123.2)
- removed the J4 at (223.0, 86.8)
- removed the J5 at (259.8, 114.3)
- removed the J6 at (259.8, 108.0)
- removed the R1 at (220.5, 62.0)
- removed the R2 at (212.8, 61.8)
- removed the U1 at (246.0, 98.6)
- removed the U2 at (237.4, 123.9)
- removed the U3 at (202.8, 61.2)
Routing:
- net I2C_SDA: track 182.9 -> 0.00 mm
- net +3V3: track 140.5 -> 0.00 mm
- net GND: track 129.0 -> 0.00 mm
- net I2C_SCL: track 127.5 -> 0.00 mm
- net +5V: track 87.0 -> 0.00 mm
- net Output_B: track 5.22 -> 0.00 mm
- net Output_A: track 5.20 -> 0.00 mm
- net Button_pin: track 5.18 -> 0.00 mm
- removed copper zone on B.Cu, net GND
